File: kicad/kint.kicad_pcb (KiCad board)
At the start: 2 copper layers, 107.9 x 86 mm, 27 parts, among them J1 THUMB_RIGHT_SPC_KB600, J2 LEFT_13_LT, J3 TOP_LEFT, J4 TOP_RIGHT, J5 THUMB_LEFT_BAK, J6 THUMB_RIGHT_SPC, J7 RIGHT_13_DOWN, J8 THUMB_LEFT_BAK_KB600, U1 TEENSY_3.5_3.6

Commit message: [WIP] playing around with promicro compatibility
Parts:
- removed JP1, JP2, JP3: SolderJumper_2_Open, Jumper:SolderJumper-2_P1.3mm_Open_RoundedPad1.0x1.5mm
- removed JP4, JP5, JP6: SolderJumper_2_Bridged, Jumper:SolderJumper-2_P1.3mm_Bridged2Bar_RoundedPad1.0x1.5mm
- removed LED1, LED2, LED3, LED4: LEDSML1206, LED_SMD:LED_1206_3216Metric_Pad1.42x1.75mm_HandSolder
- removed R1, R2, R3, R4: 10K, Resistor_SMD:R_1206_3216Metric_Pad1.42x1.75mm_HandSolder
- added D1: APA102-2020, LED_SMD:LED-APA102-2020, F.Cu at (133.3, 144.0)
- added D2: APA102-2020, LED_SMD:LED-APA102-2020, F.Cu at (143.5, 144.0)
- added D3: APA102-2020, LED_SMD:LED-APA102-2020, F.Cu at (153.6, 144.0)
- added D4: APA102-2020, LED_SMD:LED-APA102-2020, F.Cu at (163.8, 144.0)
- added U2: 74HC164, Package_SO:TSSOP-14_4.4x5mm_P0.65mm, F.Cu at (167.6, 94.0)
- added U3: 74HC164, Package_SO:TSSOP-14_4.4x5mm_P0.65mm, F.Cu at (167.6, 101.6)
- U1: value TEENSY_3.5_3.6 -> ProMicro; footprint kinx:TEENSY_3.5_3.6 -> promicro:ProMicro; moved to F.Cu
- moved U1 1.29 mm to (144.8, 101.6), turned to 0 degrees
Connections:
- U1 pad 2: /ROW_MIN -> unconnected-(U1-Pad2)
- U1 pad 24: /LED_KEYPAD -> unconnected-(U1-Pad24)
- U1 pad 5: /ROW_6 -> /LED_DATA
- U1 pad 6: /COL_6 -> /LED_CLOCK
- U1 pad 7: Net-(JP4-Pad2) -> unconnected-(U1-Pad7)
- U1 pad 8: /ROW_EQL -> unconnected-(U1-Pad8)
Routing:
- net (no net): track 0.00 -> 264.7 mm, vias 0 -> 2
- net /3V3: track 94.2 -> 0.00 mm, vias 1 -> 0
- net unconnected-(U1-Pad2): track 0.00 -> 55.0 mm, vias 0 -> 1
- net /LED_KEYPAD: track 55.0 -> 0.00 mm, vias 1 -> 0
- net unconnected-(U1-Pad8): track 0.00 -> 51.4 mm
- net /ROW_EQL: track 51.4 -> 0.00 mm
- net unconnected-(U1-Pad7): track 0.00 -> 49.9 mm
- net /ROW_1: track 49.9 -> 0.00 mm
- net unconnected-(U1-Pad1): track 0.00 -> 47.3 mm, vias 0 -> 1
- net /LED_SCROLL_LOCK: track 47.3 -> 0.00 mm, vias 1 -> 0
- net GND: track 2.54 -> 43.4 mm, vias 0 -> 1
- net /LED_CAPS_LOCK: track 40.9 -> 0.00 mm, vias 1 -> 0
- net /LED_NUM_LOCK: track 38.9 -> 0.00 mm, vias 1 -> 0
- net /ROW_9: track 80.5 -> 101.3 mm
- net /ROW_F2: track 151.9 -> 170.1 mm
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